Commit message: Updated wheel material to fix color

File: f1tarmo_description/model/robot.urdf (robot description, URDF)
Before this commit: robot model, 10 links, 9 joints
Links:
- link wheel_110mm: mass 1e-09 -> 0.2311
- link wheel_110mm_2: mass 1e-09 -> 0.2311
- link wheel_110mm_3: mass 1e-09 -> 0.2311
- link wheel_110mm_4: mass 1e-09 -> 0.2311
