Commit message: Add D435i instance to the f1tarmo parent URDF

File: f1tarmo_description/model/f1tarmo.urdf.xacro (robot description, xacro)
@@ -1,12 +1,12 @@
 <?xml version="1.0"?>
 <robot name="f1tarmo" xmlns:xacro="http://ros.org/wiki/xacro">
-    <!-- Name for RealSense camera frame -->
-    <xacro:arg name="name" default="realsense" />
-    <!-- Name of link in f1tarmo urdf that the realsense bottom screw link will
-    be mounted to -->
-    <xacro:arg name="parent" default="realsense_bottom_screw_mount" />
     <!-- Include the robot (e.g. AgileX Scout mini) -->
     <xacro:include filename="$(find f1tarmo_description)/model/robot.urdf" />
-    <!-- Add the RealSense D435i -->
+    <!-- Add the RealSense D435i xacro file. This contains a macro for creating
+    a D435i instance. -->
     <xacro:include filename="$(find realsense2_description)/urdf/_d435i.urdf.xacro"/>
+    <!-- Create a D435i instance -->
+    <xacro:sensor_d435i name="realsense" parent="realsense_bottom_screw_mount" use_nominal_extrinsics="true">
+        <origin xyz="0 0 0" rpy="-3.14 0 1.57"/>
+    </xacro:sensor_d435i>
 </robot>

Commit message: Added dummy link coincident with the drive assembly with no inertia

File: f1tarmo_description/model/f1tarmo.urdf.xacro (robot description, xacro)
@@ -1,10 +1,19 @@
 <?xml version="1.0"?>
 <robot name="f1tarmo" xmlns:xacro="http://ros.org/wiki/xacro">
-    <!-- Include the robot (e.g. AgileX Scout mini) -->
+    <!-- Include the f1tarmo base URDF generated from onshape. -->
     <xacro:include filename="$(find f1tarmo_description)/model/robot.urdf" />
+    <!-- Add a dummy parent link to the drive assembly that has zero inertia
+    (this makes KDL happy). -->
+    <link name="f1tarmo_root"/>
+    <joint name="f1tarmo_root_joint" type="fixed">
+        <parent link="f1tarmo_root"/>
+        <child link="drive_assembly"/>
+        <origin xyz="0 0 0" rpy="0 0 0"/>
+        <axis xyz="0 0 1"/>
+    </joint>
     <!-- Add the RealSense D435i xacro file. This contains a macro for creating
     a D435i instance. -->
     <xacro:include filename="$(find realsense2_description)/urdf/_d435i.urdf.xacro"/>
-    <!-- Create a D435i instance -->
+    <!-- Create a D435i instance. -->
     <xacro:sensor_d435i name="realsense" parent="realsense_bottom_screw_mount" use_nominal_extrinsics="true">
         <origin xyz="0 0 0" rpy="-3.14 0 1.57"/>
